Commit message: Update README.md

File: catkin_ws/src/minnie_description/urdf/minnie.xacro (robot description, xacro)
@@ -15,5 +15,5 @@
   </link>
   <joint name="base_link_joint" type="fixed">
-    <origin xyz="0 0 0.0635" rpy="0 0 0" />
+    <origin xyz="0 0 0.03175" rpy="0 0 0" />
     <parent link="base_footprint"/>
     <child link="base_link" />
@@ -23,5 +23,5 @@
       <origin rpy="0 1.5708 0" />
       <geometry>
-        <cylinder radius="0.0635" length="0.0254" />
+        <cylinder radius="0.03175" length="0.0254" />
       </geometry>
     </visual>
@@ -29,5 +29,5 @@
       <origin rpy="0 1.5708 0" />
       <geometry>
-        <cylinder radius="0.0635" length="0.0254" />
+        <cylinder radius="0.03175" length="0.0254" />
       </geometry>
     </collision>
@@ -42,5 +42,5 @@
       <origin rpy="0 1.5708 0" />
       <geometry>
-        <cylinder radius="0.0635" length="0.0254" />
+        <cylinder radius="0.03175" length="0.0254" />
       </geometry>
     </visual>
@@ -48,5 +48,5 @@
       <origin rpy="0 1.5708 0" />
       <geometry>
-        <cylinder radius="0.0635" length="0.0254" />
+        <cylinder radius="0.03175" length="0.0254" />
       </geometry>
     </collision>
